Commit message: doa human+

File: src/visual_filter/realtime_urdf_filter/urdf/example.urdf.xacro (robot description, xacro)
@@ -14,5 +14,5 @@
         </collision>>
     </link>
-    <link name="wall2">
+    <!-- <link name="wall2">
         <visual>
             <geometry>
@@ -25,14 +25,15 @@
             </geometry>
         </collision>>
-    </link>
+    </link> -->
     <joint name="wall1_joint" type="fixed" >
-        <origin xyz="0 1.5 0" rpy="0 0 0.785398163"/>
+        <!-- <origin xyz="0 -0.5 0" rpy="0 0 0.785398163"/> -->
+        <origin xyz="0 -0.3 0" rpy="0 0 0"/>
         <parent link="base_link"/>
         <child link="wall1"/>
     </joint>
-    <joint name="wall2_joint" type="fixed" >
-        <origin xyz="0 1.5 0" rpy="0 0 -0.785398163"/>
+    <!-- <joint name="wall2_joint" type="fixed" >
+        <origin xyz="0 -1.5 0" rpy="0 0 -0.785398163"/>
         <parent link="base_link"/>
         <child link="wall2"/>
-    </joint>
+    </joint> -->
 </robot>
